Commit message: add new node for controller

File: 40_Simulation/cs558/install/OldOne_description/share/OldOne_description/urdf/OldOne.xacro (robot description, xacro)
@@ -1,182 +1 @@
-<?xml version="1.0" ?>
-<robot name="OldOne" xmlns:xacro="http://www.ros.org/wiki/xacro">
-<xacro:include filename="$(find OldOne_description)/urdf/materials.xacro" />
-<xacro:include filename="$(find OldOne_description)/urdf/OldOne.trans" />
-<xacro:include filename="$(find OldOne_description)/urdf/OldOne.gazebo" />
-<link name="base_link">
-  <inertial>
-    <origin xyz="1.5178268510464705e-05 0.014005171546671564 0.061701996477268484" rpy="0 0 0"/>
-    <mass value="5.378132785849099"/>
-    <inertia ixx="0.010065" iyy="0.010253" izz="0.012658" ixy="-1e-06" iyz="0.000346" ixz="5e-06"/>
-  </inertial>
-  <visual>
-    <origin xyz="0 0 0" rpy="0 0 0"/>
-    <geometry>
-      <mesh filename="file://$(find OldOne_description)/meshes/base_link.stl" scale="0.001 0.001 0.001"/>
-    </geometry>
-    <material name="silver"/>
-  </visual>
-  <collision>
-    <origin xyz="0 0 0" rpy="0 0 0"/>
-    <geometry>
-      <mesh filename="file://$(find OldOne_description)/meshes/base_link.stl" scale="0.001 0.001 0.001"/>
-    </geometry>
-  </collision>
-</link>
-<link name="link1_1">
-  <inertial>
-    <origin xyz="3.635902544574233e-06 -0.010910692503208138 0.0635196732124635" rpy="0 0 0"/>
-    <mass value="12.62285791185736"/>
-    <inertia ixx="0.030809" iyy="0.027068" izz="0.026243" ixy="1e-06" iyz="0.000743" ixz="-1e-06"/>
-  </inertial>
-  <visual>
-    <origin xyz="0.0 -0.012485 -0.0989" rpy="0 0 0"/>
-    <geometry>
-      <mesh filename="file://$(find OldOne_description)/meshes/link1_1.stl" scale="0.001 0.001 0.001"/>
-    </geometry>
-    <material name="silver"/>
-  </visual>
-  <collision>
-    <origin xyz="0.0 -0.012485 -0.0989" rpy="0 0 0"/>
-    <geometry>
-      <mesh filename="file://$(find OldOne_description)/meshes/link1_1.stl" scale="0.001 0.001 0.001"/>
-    </geometry>
-  </collision>
-</link>
-<link name="link2_1">
-  <inertial>
-    <origin xyz="-4.287147710366737e-10 -0.06347856761523346 0.21249992722305178" rpy="0 0 0"/>
-    <mass value="38.297871580095894"/>
-    <inertia ixx="1.185269" iyy="1.176136" izz="0.066964" ixy="-0.0" iyz="0.0" ixz="-1.7e-05"/>
-  </inertial>
-  <visual>
-    <origin xyz="0.0 0.061915 -0.1623" rpy="0 0 0"/>
-    <geometry>
-      <mesh filename="file://$(find OldOne_description)/meshes/link2_1.stl" scale="0.001 0.001 0.001"/>
-    </geometry>
-    <material name="silver"/>
-  </visual>
-  <collision>
-    <origin xyz="0.0 0.061915 -0.1623" rpy="0 0 0"/>
-    <geometry>
-      <mesh filename="file://$(find OldOne_description)/meshes/link2_1.stl" scale="0.001 0.001 0.001"/>
-    </geometry>
-  </collision>
-</link>
-<link name="link3_1">
-  <inertial>
-    <origin xyz="-1.8938477095566052e-06 0.06111231017444019 0.16892814494444597" rpy="0 0 0"/>
-    <mass value="21.793722740171454"/>
-    <inertia ixx="0.485506" iyy="0.480773" izz="0.026538" ixy="1e-06" iyz="-0.031253" ixz="1.1e-05"/>
-  </inertial>
-  <visual>
-    <origin xyz="0.0 0.061915 -0.5873" rpy="0 0 0"/>
-    <geometry>
-      <mesh filename="file://$(find OldOne_description)/meshes/link3_1.stl" scale="0.001 0.001 0.001"/>
-    </geometry>
-    <material name="silver"/>
-  </visual>
-  <collision>
-    <origin xyz="0.0 0.061915 -0.5873" rpy="0 0 0"/>
-    <geometry>
-      <mesh filename="file://$(find OldOne_description)/meshes/link3_1.stl" scale="0.001 0.001 0.001"/>
-    </geometry>
-  </collision>
-</link>
-<link name="link4_1">
-  <inertial>
-    <origin xyz="0.0025845378830547895 -0.06207891045089357 8.053605569546818e-06" rpy="0 0 0"/>
-    <mass value="5.163345270910103"/>
-    <inertia ixx="0.006941" iyy="0.005385" izz="0.00857" ixy="0.000203" iyz="2e-06" ixz="-1e-06"/>
-  </inertial>
-  <visual>
-    <origin xyz="0.0 0.040415 -0.9795" rpy="0 0 0"/>
-    <geometry>
-      <mesh filename="file://$(find OldOne_description)/meshes/link4_1.stl" scale="0.001 0.001 0.001"/>
-    </geometry>
-    <material name="silver"/>
-  </visual>
-  <collision>
-    <origin xyz="0.0 0.040415 -0.9795" rpy="0 0 0"/>
-    <geometry>
-      <mesh filename="file://$(find OldOne_description)/meshes/link4_1.stl" scale="0.001 0.001 0.001"/>
-    </geometry>
-  </collision>
-</link>
-<link name="link5_1">
-  <inertial>
-    <origin xyz="-0.04589828597482213 -9.161157735901315e-06 -0.003949311213854112" rpy="0 0 0"/>
-    <mass value="4.252012545206828"/>
-    <inertia ixx="0.004795" iyy="0.005555" izz="0.003877" ixy="-2e-06" iyz="-1e-06" ixz="-8.4e-05"/>
-  </inertial>
-  <visual>
-    <origin xyz="0.0463 0.120815 -0.9795" rpy="0 0 0"/>
-    <geometry>
-      <mesh filename="file://$(find OldOne_description)/meshes/link5_1.stl" scale="0.001 0.001 0.001"/>
-    </geometry>
-    <material name="silver"/>
-  </visual>
-  <collision>
-    <origin xyz="0.0463 0.120815 -0.9795" rpy="0 0 0"/>
-    <geometry>
-      <mesh filename="file://$(find OldOne_description)/meshes/link5_1.stl" scale="0.001 0.001 0.001"/>
-    </geometry>
-  </collision>
-</link>
-<link name="link6_1">
-  <inertial>
-    <origin xyz="3.283135568965534e-10 3.5102179765655883e-07 0.062259568401877186" rpy="0 0 0"/>
-    <mass value="39.58468009803446"/>
-    <inertia ixx="1.450456" iyy="1.450456" izz="2.885" ixy="-0.0" iyz="1e-06" ixz="0.0"/>
-  </inertial>
-  <visual>
-    <origin xyz="0.0997 0.120815 -1.0252" rpy="0 0 0"/>
-    <geometry>
-      <mesh filename="file://$(find OldOne_description)/meshes/link6_1.stl" scale="0.001 0.001 0.001"/>
-    </geometry>
-    <material name="silver"/>
-  </visual>
-  <collision>
-    <origin xyz="0.0997 0.120815 -1.0252" rpy="0 0 0"/>
-    <geometry>
-      <mesh filename="file://$(find OldOne_description)/meshes/link6_1.stl" scale="0.001 0.001 0.001"/>
-    </geometry>
-  </collision>
-</link>
-<joint name="base_link_to_link1" type="continuous">
-  <origin xyz="0.0 0.012485 0.0989" rpy="0 0 0"/>
-  <parent link="base_link"/>
-  <child link="link1_1"/>
-  <axis xyz="0.0 0.0 1.0"/>
-</joint>
-<joint name="link1_to_link2" type="continuous">
-  <origin xyz="0.0 -0.0744 0.0634" rpy="0 0 0"/>
-  <parent link="link1_1"/>
-  <child link="link2_1"/>
-  <axis xyz="0.0 -1.0 0.0"/>
-</joint>
-<joint name="link2_to_link3" type="continuous">
-  <origin xyz="0.0 0.0 0.425" rpy="0 0 0"/>
-  <parent link="link2_1"/>
-  <child link="link3_1"/>
-  <axis xyz="-0.0 1.0 -0.0"/>
-</joint>
-<joint name="link3_to_link4" type="continuous">
-  <origin xyz="0.0 0.0215 0.3922" rpy="0 0 0"/>
-  <parent link="link3_1"/>
-  <child link="link4_1"/>
-  <axis xyz="-0.0 -1.0 0.0"/>
-</joint>
-<joint name="link4_to_link5" type="continuous">
-  <origin xyz="-0.0463 -0.0804 0.0" rpy="0 0 0"/>
-  <parent link="link4_1"/>
-  <child link="link5_1"/>
-  <axis xyz="-1.0 -0.0 -0.0"/>
-</joint>
-<joint name="link5_to_link6" type="continuous">
-  <origin xyz="-0.0534 0.0 0.0457" rpy="0 0 0"/>
-  <parent link="link5_1"/>
-  <child link="link6_1"/>
-  <axis xyz="-0.0 -0.0 1.0"/>
-</joint>
-</robot>
+/home/Gery/Marble_Balancing_Robotic_Arm/40_Simulation/cs558/build/OldOne_description/urdf/OldOne.xacro

File: 40_Simulation/cs558/install/OldOne_description/share/OldOne_description/urdf/materials.xacro (robot description, xacro)
@@ -1,6 +1 @@
-<?xml version="1.0" ?>
-<robot name="OldOne" xmlns:xacro="http://www.ros.org/wiki/xacro" >
-<material name="silver">
-  <color rgba="0.700 0.700 0.700 1.000"/>
-</material>
-</robot>
+/home/Gery/Marble_Balancing_Robotic_Arm/40_Simulation/cs558/build/OldOne_description/urdf/materials.xacro
